Commit message: update source code

File: src/d_hospital_description/urdf/d_hospital.xacro (robot description, xacro)
@@ -3,5 +3,5 @@
     <xacro:arg name="sim_mode" default="false"/>
     <xacro:include filename="ros2_control.xacro"/>
-    <!--<xacro:include filename="gazebo_control.xacro"/> -->
+    <!--<xacro:include filename="gazebo_control.xacro"/>-->
     <xacro:include filename="d_hospital_core.xacro"/>
     <xacro:include filename="camera.xacro"/>
@@ -9,5 +9,2 @@
     <xacro:include filename="lidar.xacro"/>
 </robot>
-tatic_covariance_orientation: [3.83997e-05, 0.0, 0.0, 6.46961e-05, 0.0, 0.0, 5.36936e-06, 0.0, 0.0]
-static_covariance_angular_velocity: [2.08886e-06, 0.0, 0.0, 7.21758e-05, 0.0, 0.0, 2.46344e-06, 0.0, 0.0]
-static_covariance_linear_acceleration: [0.00584827, 0.0, 0.0, 0.00387499, 0.0, 0.0, 0.0330879, 0.0, 0.0]

File: src/d_hospital_description/urdf/d_hospital_core.xacro (robot description, xacro)
@@ -21,5 +21,5 @@
   <link name="base_link">
       <visual>
-        <origin xyz="${base_length/2} 0 ${-wheel_zoff}" rpy="0 0 ${pi}"/>
+	      <origin xyz="${base_length/2} 0 ${-wheel_zoff}" rpy="0 0 ${pi/2}"/>
           <geometry>
               <mesh filename="package://d_hospital_description/meshes/robot_chassis.dae" />

File: src/d_hospital_description/urdf/lidar.xacro (robot description, xacro)
@@ -21,5 +21,5 @@
         <parent link="base_link"/>
         <child link="lidar_link"/>
-        <origin xyz="0.1385 0.0095 0.08" rpy="0 0 ${-pi/2}"/>
+	<origin xyz="0.1385 0.0095 0.08" rpy="0 0 ${pi}"/>
         <axis xyz="0 0 1"/>
     </joint>

File: src/d_hospital_description/urdf/ros2_control.xacro (robot description, xacro)
@@ -8,5 +8,5 @@
           <param name='left_wheel_name'>left_wheel_joint</param>
           <param name='right_wheel_name'>right_wheel_joint</param>
-	  <param name='enc_ticks_per_rev'>1084</param>
+	  <param name='enc_ticks_per_rev'>12</param>
           <param name='loop_rate'>30.0</param>
       </hardware>

Commit message: Corrigindo urdf

File: src/d_hospital_description/urdf/d_hospital.xacro (robot description, xacro)
@@ -5,6 +5,6 @@
     <xacro:include filename="gazebo_control.xacro"/>
     <xacro:include filename="d_hospital_core.xacro"/>
-    <xacro:include filename="camera.xacro"/>
+    <!--<xacro:include filename="camera.xacro"/>
     <xacro:include filename="imu.xacro"/>
-    <xacro:include filename="lidar.xacro"/>
+    <xacro:include filename="lidar.xacro"/>-->
 </robot>

File: src/d_hospital_description/urdf/d_hospital_core.xacro (robot description, xacro)
@@ -1,210 +1,235 @@
 <?xml version="1.0" ?>
-<robot xmlns:xacro="http://ros.org/wiki/xacro">
-  <xacro:include filename="inertial_macros.xacro"/>
-  <!-- Robot's base properties -->
-  <xacro:property name="base_length" value="0.21"/>
-  <xacro:property name="base_width" value="0.11"/>
-  <xacro:property name="base_height" value="0.035"/>
-  <!-- Robot's wheel properties -->
+<robot name="d_hospital" xmlns:xacro="http://www.ros.org/wiki/xacro">
+  <!--
+    Arquivo gerado a partir dos STLs exportados da montagem SolidWorks.
+    Convenção adotada:
+      - STLs em milímetros: mesh_scale = 0.001.
+      - Eixo X do SolidWorks -> eixo X do ROS.
+      - Eixo Y do SolidWorks -> eixo Z do ROS.
+      - Eixo Z do SolidWorks -> eixo -Y do ROS.
+      - base_link fica no centro longitudinal/lateral do chassi e na altura do eixo das rodas.
+      - base_footprint fica no solo, abaixo de base_link.
+    Coloque as malhas renomeadas em:
+      d_hospital_description/meshes/mhemapcomp_clean/
+  -->
+  <xacro:property name="mesh_dir" value="package://d_hospital_description/meshes/mhemapcomp_clean"/>
+  <xacro:property name="mesh_scale" value="0.001"/>
+  <!-- Origem da montagem SolidWorks, em metros, usada para alinhar todas as peças ao base_link. -->
+  <xacro:property name="sw_origin_x" value="0.127772"/>
+  <xacro:property name="sw_origin_y" value="0.038959"/>
+  <xacro:property name="sw_origin_z" value="0.234666"/>
+  <xacro:property name="sw_tx" value="-0.127772"/>
+  <xacro:property name="sw_ty" value="0.234666"/>
+  <xacro:property name="sw_tz" value="-0.038959"/>
+  <!-- Propriedades obtidas das dimensões dos STLs. -->
+  <xacro:property name="base_length" value="0.25"/>
+  <xacro:property name="base_width"  value="0.18"/>
+  <xacro:property name="base_height" value="0.0532"/>
+  <xacro:property name="base_mass" value="1.20"/>
+  <xacro:property name="base_collision_z" value="0.01245"/>
   <xacro:property name="wheel_radius" value="0.0325"/>
-  <xacro:property name="wheel_height" value="0.025"/>
+  <xacro:property name="wheel_width" value="0.03"/>
   <xacro:property name="wheel_mass" value="0.031"/>
-  <!-- Distance between centre of wheel and robot base -->
-  <xacro:property name="wheel_zoff" value="0.0125"/>
+  <xacro:property name="wheel_separation" value="0.1648"/>
+  <!-- Transforma uma malha exportada em coordenadas globais do SolidWorks para o frame base_link. -->
+  <xacro:macro name="solidworks_base_visual" params="visual_name mesh_file">
+    <visual name="${visual_name}">
+      <origin xyz="${sw_tx} ${sw_ty} ${sw_tz}" rpy="${pi/2} 0 0"/>
+      <geometry>
+        <mesh filename="${mesh_dir}/${mesh_file}" scale="${mesh_scale} ${mesh_scale} ${mesh_scale}"/>
+      </geometry>
+    </visual>
+  </xacro:macro>
+  <!-- Visual de uma malha cujo link está no centro da própria peça. -->
+  <xacro:macro name="solidworks_centered_visual" params="mesh_file ox oy oz">
+    <visual>
+      <origin xyz="${ox} ${oy} ${oz}" rpy="${pi/2} 0 0"/>
+      <geometry>
+        <mesh filename="${mesh_dir}/${mesh_file}" scale="${mesh_scale} ${mesh_scale} ${mesh_scale}"/>
+      </geometry>
+    </visual>
+  </xacro:macro>
   <link name="base_footprint"/>
-   <joint name="base_joint" type="fixed">
-     <parent link="base_footprint"/>
-     <child link="base_link"/>
-     <origin xyz="-0.076 0 ${(wheel_radius + wheel_zoff / 2)}" rpy="0 0 0"/>
-   </joint>
-  <!-- Robot base chasis-->
+  <joint name="base_joint" type="fixed">
+    <parent link="base_footprint"/>
+    <child link="base_link"/>
+    <origin xyz="0 0 ${wheel_radius}" rpy="0 0 0"/>
+  </joint>
   <link name="base_link">
-      <visual>
-	      <origin xyz="${base_length/2} 0 ${-wheel_zoff}" rpy="0 0 ${pi/2}"/>
-          <geometry>
-              <mesh filename="package://d_hospital_description/meshes/robot_chassis.dae" />
-          </geometry>
-      </visual>
-      <collision>
-        <origin xyz="${base_length/2} 0 ${-wheel_zoff}" rpy="0 0 0"/>
-        <geometry>
-          <box size="${base_length} ${base_width} ${base_height}"/>
-        </geometry>
-      </collision>
-    <!-- Caster mount -->
-      <visual name="caster_mount_visual">
-          <origin xyz="0.0185 0 -0.0475" rpy="0 0 0"/>
-        <geometry>
-          <mesh filename="package://d_hospital_description/meshes/caster_mount.dae" />
-        </geometry>
-      </visual>
-      <collision name="caster_mount_collision">
-        <origin xyz="0.0185 0 -0.005" rpy="0 0 0"/>
-        <geometry>
-          <cylinder radius="0.023" length="0.0125"/>
-        </geometry>
-      </collision>
-      <!-- Rpi stand -->
-      <visual name="rpi_4_stand_visual">
-        <origin xyz="0.045 0.015 0.031" rpy="${pi} 0 ${-pi}"/>
-          <geometry>
-              <mesh filename="package://d_hospital_description/meshes/rpi_stand.dae" />
-          </geometry>
-      </visual>
-      <collision name="rpi_4_stand_collision">
-        <origin xyz="0.045 0 0.017" rpy="0 0 ${pi/2}"/>
-        <geometry>
-          <box size="0.098 0.065 0.034"/>
-        </geometry>
-      </collision>
-      <!-- Raspberry Pi -->
-      <visual name="rpi_4_visual">
-        <origin xyz="0.046 0.00245 0.033" rpy="0 0 ${pi/2}"/>
-        <geometry>
-          <mesh filename="package://d_hospital_description/meshes/rpi_4.dae"/>
-        </geometry>
-      </visual>
-      <collision name="rpi_4_collision">
-        <origin xyz="0.047 0.005 0.041" rpy="0 0 ${pi/2}"/>
-        <geometry>
-          <box size="0.09 0.06 0.02"/>
-        </geometry>
-      </collision>
-      <!-- Power bank stand -->
-      <visual name="power_bank_stand_visual">
-        <origin xyz="0.138 0.015 0.031" rpy="${pi} 0 ${pi}"/>
-        <geometry>
-          <mesh filename="package://d_hospital_description/meshes/power_bank_stand.dae"/>
-        </geometry>
-      </visual>
-      <collision name="power_bank_stand_collision">
-        <origin xyz="0.138 0 0.0085" rpy="0 0 ${pi/2}"/>
-        <geometry>
-          <box size="0.098 0.065 0.015"/>
-        </geometry>
-      </collision>
-      <!-- Power bank -->
-      <visual name="power_bank_visual">
-        <origin xyz="0.1685 0.04775 0.015" rpy="0 0 ${pi/2}"/>
-        <geometry>
-          <mesh filename="package://d_hospital_description/meshes/power_bank.dae"/>
-        </geometry>
-      </visual>
-      <collision name="power_bank_collision">
-        <origin xyz="0.138 0 0.025" rpy="0 0 ${pi/2}"/>
-        <geometry>
-          <box size="0.096 0.062 0.02"/>
-        </geometry>
-      </collision>
-      <!-- Rplidar stand -->
-      <visual name="rplidar_stand_visual">
-        <origin xyz="0.138 0.015 0.017" rpy="0 0 ${-2*pi}"/>
-        <geometry>
-          <mesh filename="package://d_hospital_description/meshes/rplidar_stand.dae"/>
-        </geometry>
-      </visual>
-      <collision name="rplidar_stand_collision">
-        <origin xyz="0.138 0 0.04" rpy="0 0 ${pi/2}"/>
-        <geometry>
-          <box size="0.098 0.065 0.015"/>
-        </geometry>
-      </collision>
-      <!-- Rplidar base -->
-      <visual name="rplidar_base_visual">
-        <origin xyz="0.13985 0.0087 0.037" rpy="0 0 ${-pi/2}"/>
-          <geometry>
-            <mesh filename="package://d_hospital_description/meshes/rplidar_base.dae"/>
-          </geometry>
-        </visual>
-      <collision name="rplidar_base_collision">
-        <origin xyz="0.138 0 0.056" rpy="0 0 ${-pi/2}"/>
-        <geometry>
-          <box size="0.11 0.072 0.035"/>
-        </geometry>
-      </collision>
-      <!-- Camera mount -->
-      <visual name="camera_mount_visual">
-        <origin xyz="0.16 0.0335 0.001" rpy="0 0 ${pi}"/>
-          <geometry>
-            <mesh filename="package://d_hospital_description/meshes/rpi_camera_mount.dae"/>
-          </geometry>
-      </visual>
-      <collision name="camera_mount_collision">
-        <origin xyz="0.197 0.0 0.032" rpy="${pi/2} 0 ${pi/2}"/>
-        <geometry>
-          <box size="0.048 0.06 0.033"/>
-        </geometry>
-      </collision>
-    <xacro:box_inertia mass="0.864" length="${base_length}" width="${base_width}" height="${base_height}">
-      <origin xyz="0.105 0 0.0175" rpy="0 0 0"/>
-    </xacro:box_inertia>
-  </link>
-  <!-- Roda esquerda -->
+    <xacro:solidworks_base_visual visual_name="chassis_visual" mesh_file="chassis.stl"/>
+    <xacro:solidworks_base_visual visual_name="upper_deck_visual" mesh_file="upper_deck.stl"/>
+    <xacro:solidworks_base_visual visual_name="rear_panel_visual" mesh_file="rear_panel.stl"/>
+    <xacro:solidworks_base_visual visual_name="support_mhm_visual" mesh_file="support_mhm.stl"/>
+    <xacro:solidworks_base_visual visual_name="driver_l298n_visual" mesh_file="driver_l298n.stl"/>
+    <xacro:solidworks_base_visual visual_name="esp32_visual" mesh_file="esp32.stl"/>
+    <xacro:solidworks_base_visual visual_name="jetson_nano_visual" mesh_file="jetson_nano.stl"/>
+    <xacro:solidworks_base_visual visual_name="powerbank_visual" mesh_file="powerbank.stl"/>
+    <xacro:solidworks_base_visual visual_name="xl4015_regulator_visual" mesh_file="xl4015_regulator.stl"/>
+    <xacro:solidworks_base_visual visual_name="left_motor_visual" mesh_file="left_motor.stl"/>
+    <xacro:solidworks_base_visual visual_name="right_motor_visual" mesh_file="right_motor.stl"/>
+    <xacro:solidworks_base_visual visual_name="left_encoder_coupler_lm393_visual" mesh_file="left_encoder_coupler_lm393.stl"/>
+    <xacro:solidworks_base_visual visual_name="right_encoder_coupler_lm393_visual" mesh_file="right_encoder_coupler_lm393.stl"/>
+    <xacro:solidworks_base_visual visual_name="left_encoder_reader_visual" mesh_file="left_encoder_reader.stl"/>
+    <xacro:solidworks_base_visual visual_name="right_encoder_reader_visual" mesh_file="right_encoder_reader.stl"/>
+    <xacro:solidworks_base_visual visual_name="axis_protector_left_visual" mesh_file="axis_protector_left.stl"/>
+    <xacro:solidworks_base_visual visual_name="axis_protector_right_visual" mesh_file="axis_protector_right.stl"/>
+    <xacro:solidworks_base_visual visual_name="motor_support_01_visual" mesh_file="motor_support_01.stl"/>
+    <xacro:solidworks_base_visual visual_name="motor_support_02_visual" mesh_file="motor_support_02.stl"/>
+    <xacro:solidworks_base_visual visual_name="motor_support_03_visual" mesh_file="motor_support_03.stl"/>
+    <xacro:solidworks_base_visual visual_name="motor_support_04_visual" mesh_file="motor_support_04.stl"/>
+    <xacro:solidworks_base_visual visual_name="screw_m2_5x6_01_visual" mesh_file="screw_m2_5x6_01.stl"/>
+    <xacro:solidworks_base_visual visual_name="screw_m2_5x6_02_visual" mesh_file="screw_m2_5x6_02.stl"/>
+    <xacro:solidworks_base_visual visual_name="screw_m2_5x6_03_visual" mesh_file="screw_m2_5x6_03.stl"/>
+    <xacro:solidworks_base_visual visual_name="screw_m2_5x6_04_visual" mesh_file="screw_m2_5x6_04.stl"/>
+    <xacro:solidworks_base_visual visual_name="screw_m2_5x6_05_visual" mesh_file="screw_m2_5x6_05.stl"/>
+    <xacro:solidworks_base_visual visual_name="screw_m2_5x6_06_visual" mesh_file="screw_m2_5x6_06.stl"/>
+    <xacro:solidworks_base_visual visual_name="screw_m2_5x6_07_visual" mesh_file="screw_m2_5x6_07.stl"/>
+    <xacro:solidworks_base_visual visual_name="screw_m2_5x6_08_visual" mesh_file="screw_m2_5x6_08.stl"/>
+    <xacro:solidworks_base_visual visual_name="screw_m2_5x6_09_visual" mesh_file="screw_m2_5x6_09.stl"/>
+    <xacro:solidworks_base_visual visual_name="screw_m2_5x6_10_visual" mesh_file="screw_m2_5x6_10.stl"/>
+    <xacro:solidworks_base_visual visual_name="screw_m2_5x6_11_visual" mesh_file="screw_m2_5x6_11.stl"/>
+    <xacro:solidworks_base_visual visual_name="screw_m2_5x6_12_visual" mesh_file="screw_m2_5x6_12.stl"/>
+    <xacro:solidworks_base_visual visual_name="screw_m2_5x6_13_visual" mesh_file="screw_m2_5x6_13.stl"/>
+    <xacro:solidworks_base_visual visual_name="screw_m2_5x6_14_visual" mesh_file="screw_m2_5x6_14.stl"/>
+    <xacro:solidworks_base_visual visual_name="screw_m2_5x6_15_visual" mesh_file="screw_m2_5x6_15.stl"/>
+    <xacro:solidworks_base_visual visual_name="screw_m2_5x6_16_visual" mesh_file="screw_m2_5x6_16.stl"/>
+    <collision name="base_collision">
+      <origin xyz="0 0 ${base_collision_z}" rpy="0 0 0"/>
+      <geometry>
+        <box size="${base_length} ${base_width} ${base_height}"/>
+      </geometry>
+    </collision>
+    <inertial>
+      <origin xyz="0 0 ${base_collision_z}" rpy="0 0 0"/>
+      <mass value="${base_mass}"/>
+      <inertia
+        ixx="${(base_mass/12.0) * (base_width*base_width + base_height*base_height)}"
+        ixy="0"
+        ixz="0"
+        iyy="${(base_mass/12.0) * (base_length*base_length + base_height*base_height)}"
+        iyz="0"
+        izz="${(base_mass/12.0) * (base_length*base_length + base_width*base_width)}"/>
+    </inertial>
+  </link>
+  <!-- Roda esquerda: centro obtido diretamente do STL left_wheel.stl. -->
   <link name="left_wheel">
-    <visual>
-        <geometry>
-          <mesh filename="package://d_hospital_description/meshes/right_wheel.dae" />
-        </geometry>
-    </visual>
-    <collision>
-      <origin xyz="0 0 -0.0065" rpy="0 0 0"/>
-      <geometry>
-        <sphere radius="${wheel_radius}"/>
-      </geometry>
-    </collision>
-    <xacro:cylinder_inertia mass="${wheel_mass}" length="${wheel_height}" radius="${wheel_radius}">
-      <origin xyz="0 0 0" rpy="0 0 0"/>
-    </xacro:cylinder_inertia>
+    <xacro:solidworks_centered_visual mesh_file="left_wheel.stl" ox="-0.073522" oy="0.152366" oz="-0.038959"/>
+    <collision>
+      <origin xyz="0 0 0" rpy="${pi/2} 0 0"/>
+      <geometry>
+        <cylinder radius="${wheel_radius}" length="${wheel_width}"/>
+      </geometry>
+    </collision>
+    <inertial>
+      <origin xyz="0 0 0" rpy="0 0 0"/>
+      <mass value="${wheel_mass}"/>
+      <inertia
+        ixx="${(wheel_mass/12.0) * (3*wheel_radius*wheel_radius + wheel_width*wheel_width)}"
+        ixy="0"
+        ixz="0"
+        iyy="${0.5 * wheel_mass * wheel_radius * wheel_radius}"
+        iyz="0"
+        izz="${(wheel_mass/12.0) * (3*wheel_radius*wheel_radius + wheel_width*wheel_width)}"/>
+    </inertial>
   </link>
   <joint name="left_wheel_joint" type="continuous">
     <parent link="base_link"/>
     <child link="left_wheel"/>
-    <origin xyz="0.133 0.065 -${wheel_zoff}" rpy="-${pi/2} 0 ${pi}"/>
-    <axis xyz="0 0 -1"/>
-  </joint>
-  <!-- Roda direita -->
+    <origin xyz="-0.05425 0.0823 0" rpy="0 0 0"/>
+    <axis xyz="0 -1 0"/>
+  </joint>
+  <!-- Roda direita: centro obtido diretamente do STL right_wheel.stl. -->
   <link name="right_wheel">
-    <visual>
-      <geometry>
-        <mesh filename="package://d_hospital_description/meshes/right_wheel.dae"/>
-      </geometry>
-    </visual>
-    <collision>
-      <origin xyz="0 0 -0.0065" rpy="0 0 0"/>
-      <geometry>
-        <sphere radius="${wheel_radius}"/>
-      </geometry>
-    </collision>
-    <xacro:cylinder_inertia mass="${wheel_mass}" length="${wheel_height}" radius="${wheel_radius}">
-      <origin xyz="0 0 0" rpy="0 0 0"/>
-    </xacro:cylinder_inertia>
+    <xacro:solidworks_centered_visual mesh_file="right_wheel.stl" ox="-0.073522" oy="0.317166" oz="-0.038959"/>
+    <collision>
+      <origin xyz="0 0 0" rpy="${pi/2} 0 0"/>
+      <geometry>
+        <cylinder radius="${wheel_radius}" length="${wheel_width}"/>
+      </geometry>
+    </collision>
+    <inertial>
+      <origin xyz="0 0 0" rpy="0 0 0"/>
+      <mass value="${wheel_mass}"/>
+      <inertia
+        ixx="${(wheel_mass/12.0) * (3*wheel_radius*wheel_radius + wheel_width*wheel_width)}"
+        ixy="0"
+        ixz="0"
+        iyy="${0.5 * wheel_mass * wheel_radius * wheel_radius}"
+        iyz="0"
+        izz="${(wheel_mass/12.0) * (3*wheel_radius*wheel_radius + wheel_width*wheel_width)}"/>
+    </inertial>
   </link>
   <joint name="right_wheel_joint" type="continuous">
     <parent link="base_link"/>
     <child link="right_wheel"/>
-    <origin xyz="0.133 -0.065 -${wheel_zoff}" rpy="${pi/2} 0 ${-pi}"/>
-    <axis xyz="0 0 1"/>
-  </joint>
-  <!-- Caster wheel -->
+    <origin xyz="-0.05425 -0.0825 0" rpy="0 0 0"/>
+    <axis xyz="0 -1 0"/>
+  </joint>
+  <!-- Roda boba: mantida como junta fixa para simplificar a simulação. -->
   <link name="caster_wheel">
-    <visual>
-      <geometry>
-        <mesh filename="package://d_hospital_description/meshes/caster_wheel.dae"/>
-      </geometry>
-    </visual>
-    <collision>
-      <origin xyz="0 0 -0.001" rpy="0 0 ${pi/2}"/>
+    <xacro:solidworks_centered_visual mesh_file="caster_wheel.stl" ox="-0.224406" oy="0.234666" oz="-0.014309"/>
+    <collision>
+      <origin xyz="0 0 0" rpy="0 0 0"/>
       <geometry>
         <sphere radius="0.015"/>
       </geometry>
     </collision>
-    <xacro:sphere_inertia mass="0.033" radius="0.025">
-      <origin xyz="0 0 0" rpy="0 0 0"/>
-    </xacro:sphere_inertia>
+    <inertial>
+      <origin xyz="0 0 0" rpy="0 0 0"/>
+      <mass value="0.033"/>
+      <inertia ixx="0.00000825" ixy="0" ixz="0" iyy="0.00000825" iyz="0" izz="0.00000825"/>
+    </inertial>
   </link>
   <joint name="caster_wheel_joint" type="fixed">
     <parent link="base_link"/>
     <child link="caster_wheel"/>
-    <origin xyz="0.028 0 -0.031" rpy="0 0 ${pi/2}"/>
+    <origin xyz="0.096635 0 -0.02465" rpy="0 0 0"/>
+  </joint>
+  <!-- LIDAR: link visual separado para permitir TF do sensor. -->
+  <link name="rplidar_link">
+    <xacro:solidworks_centered_visual mesh_file="rplidar_a1.stl" ox="-0.093628" oy="0.232936" oz="-0.108759"/>
+    <collision>
+      <origin xyz="0 0 0" rpy="0 0 0"/>
+      <geometry>
+        <cylinder radius="0.050" length="0.040"/>
+      </geometry>
+    </collision>
+    <inertial>
+      <origin xyz="0 0 0" rpy="0 0 0"/>
+      <mass value="0.17"/>
+      <inertia ixx="0.00008" ixy="0" ixz="0" iyy="0.00008" iyz="0" izz="0.00012"/>
+    </inertial>
+  </link>
+  <joint name="rplidar_joint" type="fixed">
+    <parent link="base_link"/>
+    <child link="rplidar_link"/>
+    <origin xyz="-0.034144 0.001731 0.0698" rpy="0 0 0"/>
+  </joint>
+  <!-- Frame recomendado para o LaserScan. Ajuste o z se a altura real do plano do laser for medida. -->
+  <link name="laser_frame"/>
+  <joint name="laser_joint" type="fixed">
+    <parent link="rplidar_link"/>
+    <child link="laser_frame"/>
+    <origin xyz="0 0 0.020" rpy="0 0 0"/>
+  </joint>
+  <!-- IMU MPU6050: frame separado para uso com robot_localization/ekf_node. -->
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
File: src/d_hospital_description/urdf/lidar.xacro (robot description, xacro)
@@ -21,5 +21,5 @@
         <parent link="base_link"/>
         <child link="lidar_link"/>
-	<origin xyz="0.1385 0.0095 0.08" rpy="0 0 ${pi}"/>
+	<origin xyz="0.1385 0.0095 0.08" rpy="0 0 0"/>
         <axis xyz="0 0 1"/>
     </joint>
@@ -28,10 +28,10 @@
             <pose>0 0 0 0 0 0</pose>
             <always_on>true</always_on>
-            <visualize>false</visualize>
-            <update_rate>10</update_rate>
+            <visualize>true</visualize>
+            <update_rate>5</update_rate>
             <ray>
                 <scan>
                     <horizontal>
-                        <samples>360</samples>
+                        <samples>720</samples>
                         <min_angle>-3.14</min_angle>
                         <max_angle>3.14</max_angle>
@@ -39,8 +39,8 @@
                 </scan>
                 <range>
-                    <min>0.15</min>
-                    <max>6.0</max>
+                    <min>0.12</min>
+                    <max>10.0</max>
                     <!-- <max>12.0</max> -->
-                    <resolution>0.01500</resolution>
+                    <resolution>1</resolution>
 		        </range>
                 <noise>
