Commit message: adjust xacro files

File: src/d_hospital_description/urdf/d_hospital_core.xacro (robot description, xacro)
@@ -160,6 +160,6 @@
     <parent link="base_link"/>
     <child link="left_wheel"/>
-    <origin xyz="0.133 0.065 -${wheel_zoff}" rpy="-${pi/2} 0 ${pi}"/>
-    <axis xyz="0 0 -1"/>
+    <origin xyz="0.133 0.065 -${wheel_zoff}" rpy="-${pi/2} 0 0"/>
+    <axis xyz="0 0 1"/>
   </joint>
   <!-- Roda direita -->
@@ -183,5 +183,5 @@
     <parent link="base_link"/>
     <child link="right_wheel"/>
-    <origin xyz="0.133 -0.065 -${wheel_zoff}" rpy="${pi/2} 0 ${-pi}"/>
+    <origin xyz="0.133 -0.065 -${wheel_zoff}" rpy="-${pi/2} 0 0"/>
     <axis xyz="0 0 1"/>
   </joint>

File: src/d_hospital_description/urdf/imu.xacro (robot description, xacro)
@@ -12,5 +12,5 @@
     <parent link="base_link"/>
     <child link="imu_link"/>
-    <origin xyz="0.045 0 0.0175" rpy="1.57079 0 0"/>
+    <origin xyz="0.045 0 0.0175" rpy="0 0 0"/>
   </joint>
  <gazebo reference="imu_link">

Commit message: Correçao dos erros fisicos

File: src/d_hospital_description/urdf/d_hospital_core.xacro (robot description, xacro)
@@ -51,5 +51,5 @@
   <xacro:property name="wheel_width" value="0.03"/>
   <xacro:property name="wheel_mass" value="0.031"/>
-  <xacro:property name="wheel_separation" value="0.1648"/>
+  <xacro:property name="wheel_separation" value="0.165"/>
   <!-- Transforma uma malha exportada em coordenadas globais do SolidWorks para o frame base_link. -->
 <xacro:macro name="solidworks_base_visual" params="visual_name mesh_file material_name:=cinza_metalico">
@@ -176,5 +176,5 @@
     <parent link="base_link"/>
     <child link="left_wheel"/>
-    <origin xyz="-0.05425 0.0823 0" rpy="0 0 0"/>
+    <origin xyz="-0.05425 0.0825 0" rpy="0 0 0"/>
     <axis xyz="0 -1 0"/>
     </joint>

Commit message: Entregando ao mundo a branch navigation

File: src/d_hospital_description/urdf/d_hospital_core.xacro (robot description, xacro)
@@ -7,5 +7,5 @@
   <xacro:property name="base_height" value="0.035"/>
   <!-- Robot's wheel properties -->
-  <xacro:property name="wheel_radius" value="0.0325"/>
+  <xacro:property name="wheel_radius" value="0.031"/>
   <xacro:property name="wheel_height" value="0.025"/>
   <xacro:property name="wheel_mass" value="0.031"/>
@@ -59,5 +59,5 @@
       </collision>
       <!-- Raspberry Pi -->
-      <visual name="rpi_4_visual">
+      <visual name="rpi_4_visual">0
         <origin xyz="0.046 0.00245 0.033" rpy="0 0 ${pi/2}"/>
         <geometry>
@@ -148,5 +148,5 @@
     </visual>
     <collision>
-      <origin xyz="0 0 -0.0065" rpy="0 0 0"/>
+      <origin xyz="0 0 -0.0075" rpy="0 0 0"/>
       <geometry>
         <sphere radius="${wheel_radius}"/>
@@ -160,5 +160,5 @@
     <parent link="base_link"/>
     <child link="left_wheel"/>
-    <origin xyz="0.133 0.065 -${wheel_zoff}" rpy="-${pi/2} 0 0"/>
+    <origin xyz="0.133 0.075 -${wheel_zoff}" rpy="-${pi/2} 0 0"/>
     <axis xyz="0 0 1"/>
   </joint>
@@ -171,5 +171,5 @@
     </visual>
     <collision>
-      <origin xyz="0 0 -0.0065" rpy="0 0 0"/>
+      <origin xyz="0 0 -0.0075" rpy="0 0 0"/>
       <geometry>
         <sphere radius="${wheel_radius}"/>
@@ -183,5 +183,5 @@
     <parent link="base_link"/>
     <child link="right_wheel"/>
-    <origin xyz="0.133 -0.065 -${wheel_zoff}" rpy="-${pi/2} 0 0"/>
+    <origin xyz="0.133 -0.075 -${wheel_zoff}" rpy="-${pi/2} 0 0"/>
     <axis xyz="0 0 1"/>
   </joint>
