Commit message: change imu orientation

File: src/d_hospital_description/urdf/imu.xacro (robot description, xacro)
@@ -12,5 +12,5 @@
     <parent link="base_link"/>
     <child link="imu_link"/>
-    <origin xyz="0.045 0 0.0175" rpy="0 0 0"/>
+    <origin xyz="0.045 0 0.0175" rpy="1.57079 0 0"/>
   </joint>
  <gazebo reference="imu_link">
